Commit message: Update four_wheel_robot.urdf

File: four_wheel_robot.urdf (robot description, URDF)
Before this commit: robot four_wheel_service_robot, 5 links, 4 joints
Links:
- removed link front_left_wheel
- removed link front_right_wheel
- removed link rear_left_wheel
- removed link rear_right_wheel
Joints:
- removed joint front_left_wheel_joint
- removed joint front_right_wheel_joint
- removed joint rear_left_wheel_joint
- removed joint rear_right_wheel_joint
